Commit message: kuka.urdf

File: roboschool/models_robot/kuka_description/urdf/kuka.urdf (robot description, URDF)
Before this commit: robot lbr_iiwa, 8 links, 7 joints
Links:
- link lbr_iiwa_link_0: geometry collision mesh filename=package://kuka_description/meshes/link_0.stl; visual mesh filename=package://kuka_description/meshes/link_0.stl
- link lbr_iiwa_link_1: geometry collision mesh filename=package://kuka_description/meshes/link_1.stl; visual mesh filename=package://kuka_description/meshes/link_1.stl
- link lbr_iiwa_link_2: geometry collision mesh filename=package://kuka_description/meshes/link_2.stl; visual mesh filename=package://kuka_description/meshes/link_2.stl
- link lbr_iiwa_link_3: geometry collision mesh filename=package://kuka_description/meshes/link_3.stl; visual mesh filename=package://kuka_description/meshes/link_3.stl
- link lbr_iiwa_link_4: geometry collision mesh filename=package://kuka_description/meshes/link_4.stl; visual mesh filename=package://kuka_description/meshes/link_4.stl
- link lbr_iiwa_link_5: geometry collision mesh filename=package://kuka_description/meshes/link_5.stl; visual mesh filename=package://kuka_description/meshes/link_5.stl
- link lbr_iiwa_link_6: geometry collision mesh filename=package://kuka_description/meshes/link_6.stl; visual mesh filename=package://kuka_description/meshes/link_6.stl
- link lbr_iiwa_link_7: geometry collision mesh filename=package://kuka_description/meshes/link_7.stl; visual mesh filename=package://kuka_description/meshes/link_7.stl
