Commit message: corrected cuca angle limits

File: roboschool/models_robot/kuka_gripper_description/urdf/cube.urdf (robot description, URDF)
Before this commit: robot cube, 1 links, 0 joints
Links:
- link cube: mass 0.2 -> 1.0

File: roboschool/models_robot/kuka_gripper_description/urdf/kuka_gripper.urdf (robot description, URDF)
Before this commit: robot kuka_gripper, 13 links, 12 joints
Links:
- link base: mass 0.5 -> 2.0
- link finger_00: mass 0.5 -> 2.0
- link finger_01: mass 0.5 -> 2.0
- link finger_10: mass 0.5 -> 2.0
- link finger_11: mass 0.5 -> 2.0

Commit message: modified angles and masses

File: roboschool/models_robot/kuka_gripper_description/urdf/cube.urdf (robot description, URDF)
Before this commit: robot cube, 1 links, 0 joints
Links:
- link cube: mass 1.0 -> 0.6; geometry collision box size=0.06 0.06 0.06; visual box size=0.06 0.06 0.06

Commit message: colors

File: roboschool/models_robot/kuka_gripper_description/urdf/cube.urdf (robot description, URDF)
Before this commit: robot cube, 1 links, 0 joints
Links:
- removed link cube
- added link cube_0, mass 0.6; collision mesh filename=package://kuka_gripper_description/meshes/cube.obj; visual mesh filename=package://kuka_gripper_description/meshes/cube.obj
