Commit message: objects

File: roboschool/models_robot/kuka_gripper_description/urdf/tomato_soup_can.urdf (robot description, URDF)
Before this commit: robot tomato_soup_can, 1 links, 0 joints
Links:
- removed link tomato_soup_can
- added link tomato, mass 1.; collision mesh filename=package://kuka_gripper_description/meshes/tomato.obj; visual mesh filename=package://kuka_gripper_description/meshes/tomato.obj
