Commit message: working gripper

File: roboschool/models_robot/kuka_gripper_description/urdf/kuka_gripper.urdf (robot description, URDF)
Before this commit: robot lbr_iiwa, 13 links, 12 joints
Links:
- link base: geometry collision mesh filename=package://kuka_gripper_description/meshes/base.stl; visual mesh filename=package://kuka_gripper_description/meshes/base.stl
- link finger_00: geometry collision mesh filename=package://kuka_gripper_description/meshes/finger_0.stl; visual mesh filename=package://kuka_gripper_description/meshes/finger_0.stl
- link finger_01: geometry collision mesh filename=package://kuka_gripper_description/meshes/finger_1.stl; visual mesh filename=package://kuka_gripper_description/meshes/finger_1.stl
- link finger_10: geometry collision mesh filename=package://kuka_gripper_description/meshes/finger_0.stl; visual mesh filename=package://kuka_gripper_description/meshes/finger_0.stl
- link finger_11: geometry collision mesh filename=package://kuka_gripper_description/meshes/finger_1.stl; visual mesh filename=package://kuka_gripper_description/meshes/finger_1.stl
Joints:
- joint base_to_finger00_joint: origin xyz=0.023510971786833857 0 0 rpy=0 0 0 -> xyz=0.043510971786833857 0 0 rpy=0 0 0
- joint base_to_finger10_joint: origin xyz=-0.023510971786833857 0 0 rpy=0 0 3.141592653589793 -> xyz=-0.043510971786833857 0 0 rpy=0 0 3.141592653589793

Commit message: added table object to kuka_gripper

File: roboschool/models_robot/kuka_gripper_description/urdf/kuka_gripper.urdf (robot description, URDF)
Before this commit: robot lbr_iiwa, 13 links, 12 joints
Links:
- link lbr_iiwa_link_0: geometry collision mesh filename=package://kuka_gripper_description/meshes/link_0.stl; visual mesh filename=package://kuka_gripper_description/meshes/link_0.stl
- link lbr_iiwa_link_1: geometry collision mesh filename=package://kuka_gripper_description/meshes/link_1.stl; visual mesh filename=package://kuka_gripper_description/meshes/link_1.stl
- link lbr_iiwa_link_2: geometry collision mesh filename=package://kuka_gripper_description/meshes/link_2.stl; visual mesh filename=package://kuka_gripper_description/meshes/link_2.stl
- link lbr_iiwa_link_3: geometry collision mesh filename=package://kuka_gripper_description/meshes/link_3.stl; visual mesh filename=package://kuka_gripper_description/meshes/link_3.stl
- link lbr_iiwa_link_4: geometry collision mesh filename=package://kuka_gripper_description/meshes/link_4.stl; visual mesh filename=package://kuka_gripper_description/meshes/link_4.stl
- link lbr_iiwa_link_5: geometry collision mesh filename=package://kuka_gripper_description/meshes/link_5.stl; visual mesh filename=package://kuka_gripper_description/meshes/link_5.stl
- link lbr_iiwa_link_6: geometry collision mesh filename=package://kuka_gripper_description/meshes/link_6.stl; visual mesh filename=package://kuka_gripper_description/meshes/link_6.stl
- link lbr_iiwa_link_7: geometry collision mesh filename=package://kuka_gripper_description/meshes/link_7.stl; visual mesh filename=package://kuka_gripper_description/meshes/link_7.stl
Joints:
- joint kuka_to_gripper_joint: origin xyz=0 0 0.02 rpy=0 0 0 -> xyz=0 0 0.05 rpy=0 0 0

Commit message: kuka_touch

File: roboschool/models_robot/kuka_gripper_description/urdf/kuka_gripper.urdf (robot description, URDF)
Before this commit: robot kuka_gripper, 13 links, 12 joints
Links:
- link base: mass 0.03 -> 0.5
- link finger_00: mass 0.03 -> 0.5
- link finger_01: mass 0.03 -> 0.5
- link finger_10: mass 0.03 -> 0.5
- link finger_11: mass 0.03 -> 0.5

Commit message: textures and grasp

File: roboschool/models_robot/kuka_gripper_description/urdf/kuka_gripper.urdf (robot description, URDF)
Before this commit: robot kuka_gripper, 13 links, 12 joints
Links:
- link lbr_iiwa_link_0: mass 0.0 -> 0

File: roboschool/models_robot/kuka_gripper_description/urdf/table.urdf (robot description, URDF)
Before this commit: robot table, 1 links, 0 joints
Links:
- link table_0: geometry collision mesh filename=package://kuka_gripper_description/meshes/table.obj; visual mesh filename=package://kuka_gripper_description/meshes/table.obj

Commit message: objects

File: roboschool/models_robot/kuka_gripper_description/urdf/kuka_gripper.urdf (robot description, URDF)
Before this commit: robot kuka_gripper, 13 links, 12 joints
Links:
- link base: geometry collision mesh filename=package://kuka_gripper_description/meshes/base.obj; visual mesh filename=package://kuka_gripper_description/meshes/base.obj
- link finger_00: geometry collision mesh filename=package://kuka_gripper_description/meshes/finger_0.obj; visual mesh filename=package://kuka_gripper_description/meshes/finger_0.obj
- link finger_01: geometry collision mesh filename=package://kuka_gripper_description/meshes/finger_1.obj; visual mesh filename=package://kuka_gripper_description/meshes/finger_1.obj
- link finger_10: geometry collision mesh filename=package://kuka_gripper_description/meshes/finger_0.obj; visual mesh filename=package://kuka_gripper_description/meshes/finger_0.obj
- link finger_11: geometry collision mesh filename=package://kuka_gripper_description/meshes/finger_1.obj; visual mesh filename=package://kuka_gripper_description/meshes/finger_1.obj
- link lbr_iiwa_link_0: geometry collision mesh filename=package://kuka_gripper_description/meshes/link_0.obj; visual mesh filename=package://kuka_gripper_description/meshes/link_0.obj
- link lbr_iiwa_link_1: geometry collision mesh filename=package://kuka_gripper_description/meshes/link_1.obj; visual mesh filename=package://kuka_gripper_description/meshes/link_1.obj
- link lbr_iiwa_link_2: geometry collision mesh filename=package://kuka_gripper_description/meshes/link_2.obj; visual mesh filename=package://kuka_gripper_description/meshes/link_2.obj
- link lbr_iiwa_link_3: geometry collision mesh filename=package://kuka_gripper_description/meshes/link_3.obj; visual mesh filename=package://kuka_gripper_description/meshes/link_3.obj
- link lbr_iiwa_link_4: geometry collision mesh filename=package://kuka_gripper_description/meshes/link_4.obj; visual mesh filename=package://kuka_gripper_description/meshes/link_4.obj
- link lbr_iiwa_link_5: geometry collision mesh filename=package://kuka_gripper_description/meshes/link_5.obj; visual mesh filename=package://kuka_gripper_description/meshes/link_5.obj
- link lbr_iiwa_link_6: geometry collision mesh filename=package://kuka_gripper_description/meshes/link_6.obj; visual mesh filename=package://kuka_gripper_description/meshes/link_6.obj
- link lbr_iiwa_link_7: geometry collision mesh filename=package://kuka_gripper_description/meshes/link_7.obj; visual mesh filename=package://kuka_gripper_description/meshes/link_7.obj

Commit message: objects

File: roboschool/models_robot/kuka_gripper_description/urdf/kuka_gripper.urdf (robot description, URDF)
Before this commit: robot kuka_gripper, 13 links, 12 joints
Links:
- link base: geometry collision mesh filename=package://kuka_gripper_description/meshes/base.stl; visual mesh filename=package://kuka_gripper_description/meshes/base.stl
- link finger_00: geometry collision mesh filename=package://kuka_gripper_description/meshes/finger_0.stl; visual mesh filename=package://kuka_gripper_description/meshes/finger_0.stl
- link finger_01: geometry collision mesh filename=package://kuka_gripper_description/meshes/finger_1.stl; visual mesh filename=package://kuka_gripper_description/meshes/finger_1.stl
- link finger_10: geometry collision mesh filename=package://kuka_gripper_description/meshes/finger_0.stl; visual mesh filename=package://kuka_gripper_description/meshes/finger_0.stl
- link finger_11: geometry collision mesh filename=package://kuka_gripper_description/meshes/finger_1.stl; visual mesh filename=package://kuka_gripper_description/meshes/finger_1.stl
- link lbr_iiwa_link_0: geometry collision mesh filename=package://kuka_gripper_description/meshes/link_0.stl; visual mesh filename=package://kuka_gripper_description/meshes/link_0.stl
- link lbr_iiwa_link_1: geometry collision mesh filename=package://kuka_gripper_description/meshes/link_1.stl; visual mesh filename=package://kuka_gripper_description/meshes/link_1.stl
- link lbr_iiwa_link_2: geometry collision mesh filename=package://kuka_gripper_description/meshes/link_2.stl; visual mesh filename=package://kuka_gripper_description/meshes/link_2.stl
- link lbr_iiwa_link_3: geometry collision mesh filename=package://kuka_gripper_description/meshes/link_3.stl; visual mesh filename=package://kuka_gripper_description/meshes/link_3.stl
- link lbr_iiwa_link_4: geometry collision mesh filename=package://kuka_gripper_description/meshes/link_4.stl; visual mesh filename=package://kuka_gripper_description/meshes/link_4.stl
- link lbr_iiwa_link_5: geometry collision mesh filename=package://kuka_gripper_description/meshes/link_5.stl; visual mesh filename=package://kuka_gripper_description/meshes/link_5.stl
- link lbr_iiwa_link_6: geometry collision mesh filename=package://kuka_gripper_description/meshes/link_6.stl; visual mesh filename=package://kuka_gripper_description/meshes/link_6.stl
- link lbr_iiwa_link_7: geometry collision mesh filename=package://kuka_gripper_description/meshes/link_7.stl; visual mesh filename=package://kuka_gripper_description/meshes/link_7.stl
